Commit message: Add convexified objs for collision geometry

File: examples/hsr/models/urdfs/hsrb4s_coll.obj.urdf (robot description, URDF)
Before this commit: robot hsrb, 45 links, 44 joints
Joints:
- joint base_l_passive_wheel_x_frame_joint: type fixed -> continuous
- joint base_l_passive_wheel_y_frame_joint: type fixed -> continuous
- joint base_l_passive_wheel_z_joint: type fixed -> continuous
- joint base_r_passive_wheel_x_frame_joint: type fixed -> continuous
- joint base_r_passive_wheel_y_frame_joint: type fixed -> continuous
- joint base_r_passive_wheel_z_joint: type fixed -> continuous
- joint hand_l_distal_joint: type fixed -> revolute
- joint hand_l_mimic_distal_joint: type fixed -> revolute
- joint hand_l_proximal_joint: type fixed -> revolute
- joint hand_r_distal_joint: type fixed -> revolute
- joint hand_r_mimic_distal_joint: type fixed -> revolute
- joint hand_r_proximal_joint: type fixed -> revolute
- joint torso_lift_joint: type fixed -> prismatic
